File: Hardware/KiCad/picture_frame_carrier_board/picture_frame_carrier_board.kicad_sch (KiCad schematic)
At the start: 60 parts, among them J1 Conn_01x14_Socket, J10 JST-PH RM2, J2 Conn_01x18_Socket, J3 Conn_02x20_Odd_Even, J4 Conn_01x08_Socket, J5 Conn_01x08_Socket, J6 JST-PH RM2, J8 JST-PH RM2, J9 JST-PH RM2, Q1 BSH205G2AR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

Commit message: changed files
Parts:
- R1, R14, R2, R6: value 10k -> 100k
- R10, R15: value 1k -> 22k
- R21, R23, R25: value DNP -> 100k
Changed lines of the file:
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@@
       (effects (font (size 1.27 1.27)) (justify left))
     )
-    (property "Value" "10k" (at 342.9 212.725 0)
+    (property "Value" "100k" (at 342.9 212.725 0)
       (effects (font (size 1.27 1.27)) (justify left))
     )
@@
       (effects (font (size 1.27 1.27)) (justify left))
     )
-    (property "Value" "DNP" (at 78.74 96.52 90)
+    (property "Value" "100k" (at 78.74 96.52 90)
       (effects (font (size 1.27 1.27)) (justify left))
     )
@@
       (effects (font (size 1.27 1.27)) (justify left))
     )
-    (property "Value" "10k" (at 209.55 211.455 0)
+    (property "Value" "100k" (at 209.55 211.455 0)
       (effects (font (size 1.27 1.27)) (justify left))
     )
@@
       (effects (font (size 1.27 1.27)) (justify left))
     )
-    (property "Value" "10k" (at 193.04 234.315 0)
+    (property "Value" "100k" (at 193.04 234.315 0)
       (effects (font (size 1.27 1.27)) (justify left))
     )
@@
       (effects (font (size 1.27 1.27)) (justify left))
     )
-    (property "Value" "10k" (at 264.16 212.725 0)
+    (property "Value" "100k" (at 264.16 212.725 0)
       (effects (font (size 1.27 1.27)) (justify left))
     )
@@
       (effects (font (size 1.27 1.27)) (justify left))
     )
-    (property "Value" "1k" (at 365.76 220.345 0)
+    (property "Value" "22k" (at 365.76 220.345 0)
       (effects (font (size 1.27 1.27)) (justify left))
     )
@@
       (effects (font (size 1.27 1.27)) (justify left))
     )
-    (property "Value" "1k" (at 287.02 220.345 0)
+    (property "Value" "22k" (at 287.02 220.345 0)
       (effects (font (size 1.27 1.27)) (justify left))
     )
@@
       (effects (font (size 1.27 1.27)) (justify left))
     )
-    (property "Value" "DNP" (at 52.07 96.52 90)
+    (property "Value" "100k" (at 52.07 96.52 90)
       (effects (font (size 1.27 1.27)) (justify left))
     )
@@
       (effects (font (size 1.27 1.27)) (justify left))
     )
-    (property "Value" "DNP" (at 64.77 96.52 90)
-      (effects (font (size 1.27 1.27)) (justify left))
-    )
+    (property "Value" "100k" (at 64.77 96.52 90)
+      (effects (font (size 1.27 1.27)) (justify left))
+    )
